File: pcb/sensors.kicad_sch (KiCad schematic)
At the start: 0 parts

Commit message: Updated license and implemented RP2040
Parts:
- added U3: HDC1080, CRG Makes:PWSON-N6, symbol CRG Makes:HDC1080
- added U4: LTR-303ALS-01, CRG Makes:LTR-303ALS-01, symbol CRG Makes:LTR-303ALS-01
Connections:
- new net +3.3V: U3.5 (VCC), U4.1 (VDD)
- new net GND: U3.2 (GND), U4.3 (GND)
- new net SCL_INT: U3.6 (SCL), U4.4 (SCL)
- new net SDA_INT: U3.1 (SDA), U4.6 (SDA)
- no-connect marks 0 -> 1
