File: pcb/env-module.kicad_sch (KiCad schematic)
At the start: 8 parts

Commit message: Change schematic name
Other:
- title: Environment Module -> Client
Changed lines of the file:
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@@
 	(paper "A4")
 	(title_block
-		(title "Environment Module")
+		(title "Client")
 		(date "<<release-date>>")
 		(rev "<<tag>>")
