File: pcb/aquarius-client-hw.kicad_sch (KiCad schematic)
At the start: 8 parts

Commit message: Updated project name and properties
Other:
- title: Client -> Client Hardware
Changed lines of the file:
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@@
 	(paper "A4")
 	(title_block
-		(title "Client")
+		(title "Client Hardware")
 		(date "<<release-date>>")
 		(rev "<<tag>>")
@@
 		)
 		(instances
-			(project "env-module"
+			(project "aquarius-client-hw"
 				(path "/445c1fff-2e1a-48b1-a91f-a137832edebf"
 					(page "4")
@@
 		)
 		(instances
-			(project "env-module"
+			(project "aquarius-client-hw"
 				(path "/445c1fff-2e1a-48b1-a91f-a137832edebf"
 					(page "5")
@@
 		)
 		(instances
-			(project "env-module"
+			(project "aquarius-client-hw"
 				(path "/445c1fff-2e1a-48b1-a91f-a137832edebf"
 					(page "3")
@@
 		)
 		(instances
-			(project "env-module"
+			(project "aquarius-client-hw"
 				(path "/445c1fff-2e1a-48b1-a91f-a137832edebf"
 					(page "2")
@@
 		)
 		(instances
-			(project "env-module"
+			(project "aquarius-client-hw"
 				(path "/445c1fff-2e1a-48b1-a91f-a137832edebf"
 					(page "6")
@@
 		)
 		(instances
-			(project "env-module"
+			(project "aquarius-client-hw"
 				(path "/445c1fff-2e1a-48b1-a91f-a137832edebf"
 					(page "7")
