File: pcb/aquarius-client-hw.kicad_pcb (KiCad board)
At the start: 4 copper layers, 50 x 50 mm, 161 parts, among them J3 USB_C_USB2.0_16P, J4 BM03B-SRSS-TB, J9 BM08B-SRSS-TB, SW1 EVQ-Q2B02W, SW2 EVQ-Q2B02W, U1 ESP32-S3-WROOM-1-N8R2, U2 HDC1080, U3 LTR-303ALS-01, U4 USBLC6-2P6, U5 LM66200DRLR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

Commit message: Added labels for LEDs
Parts:
- added kibuzzard-689AB7E6: G***, kibuzzard-689AB7E6, F.Cu at (87.8, 86.8)
- added kibuzzard-689AB7F0: G***, kibuzzard-689AB7F0, F.Cu at (97.9, 86.8)
- added kibuzzard-689AB803: G***, kibuzzard-689AB803, F.Cu at (91.2, 86.8)
- added kibuzzard-689AB80B: G***, kibuzzard-689AB80B, F.Cu at (94.8, 86.8)
