File: pcb/aquarius-client-hw.kicad_pcb (KiCad board)
At the start: 4 copper layers, 50 x 50 mm, 165 parts, among them J3 USB_C_USB2.0_16P, J4 BM03B-SRSS-TB, J9 BM08B-SRSS-TB, SW1 EVQ-Q2B02W, SW2 EVQ-Q2B02W, U1 ESP32-S3-WROOM-1-N8R2, U2 HDC1080, U3 LTR-303ALS-01, U4 USBLC6-2P6, U5 LM66200DRLR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

Commit message: Switch cap/res to CRGM footprint
Parts:
- C1, C10, C11, C12, C13, C14, C15, C16, C2, C3, C4, C5, C6, C7, C8, C9: footprint Capacitor_SMD:C_0603_1608Metric -> CRGM Passive:C_0603_1608Metric
- R1, R2, R3, R4, R5, R6, R8, R9: footprint Resistor_SMD:R_0603_1608Metric -> CRGM Passive:R_0603_1608Metric
