File: pcb/mcu.kicad_sch (KiCad schematic)
At the start: 21 parts, among them J3 USB_C_USB2.0_16P, SW1 EVQ-Q2B02W, SW2 EVQ-Q2B02W, U1 ESP32-S3-WROOM-1-N8R2, U4 USBLC6-2P6

Commit message: Change schematic name
Other:
- title: Environment Module -> Client
Changed lines of the file:
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@@
 	(paper "A4")
 	(title_block
-		(title "Environment Module")
+		(title "Client")
 		(date "<<release-date>>")
 		(rev "<<tag>>")
@@
 			(at 110.49 36.83 0)
 			(effects
+				(font
+					(size 1.27 1.27)
+				)
+				(hide yes)
+			)
+		)
+		(property "LCSC" ""
+			(at 110.49 36.83 0)
+			(effects
+				(font
+					(size 1.27 1.27)
+				)
+				(hide yes)
+			)
+		)
+		(property "Digikey" ""
+			(at 110.49 36.83 0)
+			(effects
+				(font
+					(size 1.27 1.27)
+				)
+				(hide yes)
+			)
+		)
+		(property "Mouser" ""
+			(at 110.49 36.83 0)
+			(effects

Commit message: Updated project name and properties
Other:
- title: Client -> Client Hardware
Changed lines of the file:
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@@
 	(paper "A4")
 	(title_block
-		(title "Client")
+		(title "Client Hardware")
 		(date "<<release-date>>")
 		(rev "<<tag>>")

Commit message: Switch cap/res to CRGM footprint
Parts:
- C1, C2, C3, C4, C5, C6: footprint Capacitor_SMD:C_0603_1608Metric -> CRGM Passive:C_0603_1608Metric
- R1, R4, R5: footprint Resistor_SMD:R_0603_1608Metric -> CRGM Passive:R_0603_1608Metric
Changed lines of the file:
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@@
 			)
 		)
-		(property "Footprint" "Capacitor_SMD:C_0603_1608Metric"
+		(property "Footprint" "CRGM Passive:C_0603_1608Metric"
 			(at 73.3552 128.27 0)
 			(effects
@@
 			)
 		)
-		(property "Footprint" "Capacitor_SMD:C_0603_1608Metric"
+		(property "Footprint" "CRGM Passive:C_0603_1608Metric"
 			(at 200.3552 54.61 0)
 			(effects
@@
 			)
 		)
-		(property "Footprint" "Capacitor_SMD:C_0603_1608Metric"
+		(property "Footprint" "CRGM Passive:C_0603_1608Metric"
 			(at 119.0752 36.83 0)
 			(effects
@@
 			)
 		)
-		(property "Footprint" "Resistor_SMD:R_0603_1608Metric"
+		(property "Footprint" "CRGM Passive:R_0603_1608Metric"
 			(at 27.686 113.284 90)
 			(effects
@@
 			)
 		)
-		(property "Footprint" "Capacitor_SMD:C_0603_1608Metric"
+		(property "Footprint" "CRGM Passive:C_0603_1608Metric"
 			(at 27.6352 127 0)
 			(effects
@@
 			)
 		)
-		(property "Footprint" "Resistor_SMD:R_0603_1608Metric"
+		(property "Footprint" "CRGM Passive:R_0603_1608Metric"
 			(at 191.516 51.054 90)
 			(effects
@@
 			)
 		)
-		(property "Footprint" "Capacitor_SMD:C_0603_1608Metric"
+		(property "Footprint" "CRGM Passive:C_0603_1608Metric"
 			(at 111.4552 36.83 0)
 			(effects
@@
 			)
 		)
-		(property "Footprint" "Capacitor_SMD:C_0603_1608Metric"
+		(property "Footprint" "CRGM Passive:C_0603_1608Metric"
 			(at 33.9852 127 0)
 			(effects
@@
 			)
 		)
-		(property "Footprint" "Resistor_SMD:R_0603_1608Metric"
+		(property "Footprint" "CRGM Passive:R_0603_1608Metric"
 			(at 183.896 51.054 90)
 			(effects

Commit message: Added button inputs and pull ups
Parts:
- added R10, R11, R12, R7: 10K, Resistor_SMD:R_0603_1608Metric, symbol Device:R_US
Connections:
- net +3.3V: now also R10.1, R11.1, R12.1, R7.1
- net ADC1: now also U1.38 (IO2); no longer U1.39 (IO1)
- net ADC2: now also U1.39 (IO1); no longer U1.38 (IO2)
- net BTN2: now reaches U1.24 (IO47)
- net BTN2: now also R10.2
- net BTN1: now reaches U1.25 (IO48)
- net BTN1: now also R7.2
- net BTN3: now reaches U1.34 (IO41)
- net BTN3: now also R12.2
- net BTN4: now reaches U1.35 (IO42)
- net BTN4: now also R11.2
- no-connect marks 15 -> 11
Other:
- moved on the sheet: C6, R4, R5, TP10, TP6, TP7, TP8, TP9, U4

Commit message: Added renders and aligned connectors
Added renders
Aligned connectors to grid
Added dimensions
Fixed part numbers and values
Parts:
- C1: Tolerance (none) -> 10%
- C2: Digikey (none) -> 1276-1005-2-ND; LCSC C15849 -> C66501; MPN CL10A105KB8NNNC -> CL10B104KO8NNNC; Mouser (none) -> 187-CL10B104KO8NNNC
- R10, R11, R12, R7: footprint Resistor_SMD:R_0603_1608Metric -> CRGM Passive:R_0603_1608Metric
- U1: MPN (none) -> ESP32-S3-WROOM-1-N8R2
- U4: footprint Package_TO_SOT_SMD:SOT-666 -> CRGM Passive:SOT-666
Other:
- title: Client Hardware -> Client
Changed lines of the file:
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@@
 	(paper "A4")
 	(title_block
-		(title "Client Hardware")
+		(title "Client")
 		(date "<<release-date>>")
 		(rev "<<tag>>")
@@
 			)
 		)
-		(property "Footprint" "Resistor_SMD:R_0603_1608Metric"
+		(property "Footprint" "CRGM Passive:R_0603_1608Metric"
 			(at 125.476 62.484 90)
 			(effects
@@
 			)
 		)
-		(property "Footprint" "Package_TO_SOT_SMD:SOT-666"
+		(property "Footprint" "CRGM Passive:SOT-666"
 			(at 247.396 47.371 0)
 			(effects
@@
 			)
 		)
-		(property "Footprint" "Resistor_SMD:R_0603_1608Metric"
+		(property "Footprint" "CRGM Passive:R_0603_1608Metric"
 			(at 119.126 62.484 90)
 			(effects
@@
 			)
 		)
-		(property "MPN" "CL10A105KB8NNNC"
+		(property "MPN" "CL10B104KO8NNNC"
+			(at 118.11 33.02 0)
+			(effects
+				(font
+					(size 1.27 1.27)
+				)
+				(hide yes)
+			)
+		)
+		(property "LCSC" "C66501"
+			(at 118.11 33.02 0)
+			(effects
+				(font
+					(size 1.27 1.27)
+				)
+				(hide yes)
+			)
+		)
+		(property "Digikey" "1276-1005-2-ND"
 			(at 118.11 33.02 0)
 			(effects
@@
 			)
 		)
-		(property "LCSC" "C15849"
+		(property "Mouser" "187-CL10B104KO8NNNC"
 			(at 118.11 33.02 0)
 			(effects
@@
 			)
 		)
-		(property "Footprint" "Resistor_SMD:R_0603_1608Metric"
+		(property "Footprint" "CRGM Passive:R_0603_1608Metric"
 			(at 106.426 62.484 90)
 			(effects
@@
 			)
 		)
+		(property "Tolerance" "10%"
+			(at 110.49 33.02 0)
+			(effects
+				(font
+					(size 1.27 1.27)
+				)
+				(hide yes)
+			)
+		)
 		(pin "1"
 		)
@@
 			)
 		)
+		(property "MPN" "ESP32-S3-WROOM-1-N8R2"
+			(at 62.23 58.42 0)
+			(effects
+				(font
+					(size 1.27 1.27)
+				)
+				(hide yes)
+			)
+		)
 		(pin "5"
 		)
@@
 			)
 		)
-		(property "Footprint" "Resistor_SMD:R_0603_1608Metric"
+		(property "Footprint" "CRGM Passive:R_0603_1608Metric"
 			(at 112.776 62.484 90)
 			(effects
