File: pcb/mcu.kicad_sch (KiCad schematic)
At the start: 30 parts, among them J3 USB_C_USB2.0_16P, Q1 MMBT2222A, SW1 EVQ-Q2B02W, SW2 EVQ-Q2B02W, U1 ESP32-S3-WROOM-1-N8R2, U4 USBLC6-2P6

Commit message: Updated part attributes for consistency
Parts:
- C13, C2, C4, C5, C6, C8: Tolerance (none) -> 10%
- R1, R13: Tolerance (none) -> 5%
- R4, R5: Digikey 118-CR0603-JW-512ELFTR-ND -> CR0603-JW-512ELFTR-ND; Tolerance (none) -> 5%
Changed lines of the file:
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@@
 			)
 		)
+		(property "Tolerance" "10%"
+			(at 72.39 124.46 0)
+			(effects
+				(font
+					(size 1.27 1.27)
+				)
+				(hide yes)
+			)
+		)
 		(pin "1"
 		)
@@
 			)
 		)
+		(property "Tolerance" "10%"
+			(at 219.71 50.8 0)
+			(effects
+				(font
+					(size 1.27 1.27)
+				)
+				(hide yes)
+			)
+		)
 		(pin "1"
 		)
@@
 			)
 		)
+		(property "Tolerance" "10%"
+			(at 142.24 90.17 0)
+			(effects
+				(font
+					(size 1.27 1.27)
+				)
+				(hide yes)
+			)
+		)
 		(pin "1"
 		)
@@
 			)
 		)
+		(property "Tolerance" "10%"
+			(at 223.52 101.6 0)
+			(effects
+				(font
+					(size 1.27 1.27)
+				)
+				(hide yes)
+			)
+		)
 		(pin "1"
 		)
@@
 			)
 		)
-		(property "Datasheet" "~"
+		(property "Datasheet" "https://bourns.com/docs/product-datasheets/cr.pdf?sfvrsn=574d41f6_14"
 			(at 26.67 113.03 0)
 			(effects
@@
 			)
 		)
+		(property "Tolerance" "5%"
+			(at 26.67 113.03 0)
+			(effects
+				(font
+					(size 1.27 1.27)
+				)
+				(hide yes)
+			)
+		)
 		(pin "2"
 		)
@@
 			)
 		)
-		(property "Datasheet" "~"
+		(property "Datasheet" "https://bourns.com/docs/product-datasheets/cr.pdf?sfvrsn=574d41f6_14"
 			(at 210.82 50.8 0)
 			(effects
@@
 			)
 		)
-		(property "Description" "Resistor, US symbol"
+		(property "Description" "Thick Film Resistors - SMD 1/10Watt 5.1Kohms 5%"
 			(at 210.82 50.8 0)
 			(effects
@@
 			)
 		)
-		(property "Digikey" "118-CR0603-JW-512ELFTR-ND"
+		(property "Digikey" "CR0603-JW-512ELFTR-ND"
 			(at 210.82 50.8 0)
 			(effects
@@
 			)
 		)
+		(property "Tolerance" "5%"
+			(at 210.82 50.8 0)
+			(effects
+				(font
+					(size 1.27 1.27)
+				)
+				(hide yes)
+			)
+		)
 		(pin "2"
 		)
@@
 			)
 		)
+		(property "Tolerance" "10%"
+			(at 139.7 118.11 0)
+			(effects
+				(font
+					(size 1.27 1.27)
+				)
+				(hide yes)
+			)
+		)
 		(pin "1"
 		)
@@
 			)
 		)
-		(property "Datasheet" "https://www.vishay.com/docs/20035/dcrcwe3.pdf"
+		(property "Datasheet" "https://bourns.com/docs/product-datasheets/cr.pdf?sfvrsn=574d41f6_14"
 			(at 177.8 120.65 0)
 			(effects
@@
 			)
 		)
+		(property "Tolerance" "5%"
+			(at 177.8 120.65 90)
+			(effects
+				(font
+					(size 1.27 1.27)
+				)
+				(hide yes)
+			)
+		)
 		(pin "2"
 		)
@@
 			)
 		)
+		(property "Tolerance" "10%"
+			(at 33.02 123.19 0)
+			(effects
+				(font
+					(size 1.27 1.27)
+				)
+				(hide yes)
+			)
+		)
 		(pin "2"
 		)
@@
 			)
 		)
-		(property "Datasheet" "~"
+		(property "Datasheet" "https://bourns.com/docs/product-datasheets/cr.pdf?sfvrsn=574d41f6_14"
 			(at 203.2 50.8 0)
 			(effects
@@
 			)
 		)
-		(property "Description" "Resistor, US symbol"
+		(property "Description" "Thick Film Resistors - SMD 1/10Watt 5.1Kohms 5%"
 			(at 203.2 50.8 0)
 			(effects
@@
 			)
 		)
-		(property "Digikey" "118-CR0603-JW-512ELFTR-ND"
+		(property "Digikey" "CR0603-JW-512ELFTR-ND"
 			(at 203.2 50.8 0)
 			(effects
@@
 			(at 203.2 50.8 0)
 			(effects
+				(font
+					(size 1.27 1.27)
+				)
+				(hide yes)
+			)
+		)
+		(property "Tolerance" "5%"
+			(at 203.2 50.8 0)
+			(effects
