File: pcb/indicators.kicad_sch (KiCad schematic)
At the start: 4 parts

Commit message: Change schematic name
Parts:
- added C13, C14, C15, C16: 0.1uF, Capacitor_SMD:C_0603_1608Metric, symbol Device:C
- D1, D2, D3, D4: footprint LED_SMD:LED_WS2812B-2020_PLCC4_2.0x2.0mm -> CRGM Passive:LED_WS2812B-2020_PLCC4_2.0x2.0mm
Connections:
- net +3.3V: now also C13.1, C14.1, C15.1, C16.1
- net GND: now also C13.2, C14.2, C15.2, C16.2
Other:
- title: Environment Module -> Client

Commit message: Updated project name and properties
Other:
- title: Client -> Client Hardware
Changed lines of the file:
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@@
 	(paper "A4")
 	(title_block
-		(title "Client")
+		(title "Client Hardware")
 		(date "<<release-date>>")
 		(rev "<<tag>>")

Commit message: Switch cap/res to CRGM footprint
Parts:
- C13, C14, C15, C16: footprint Capacitor_SMD:C_0603_1608Metric -> CRGM Passive:C_0603_1608Metric
Changed lines of the file:
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@@
 			)
 		)
-		(property "Footprint" "Capacitor_SMD:C_0603_1608Metric"
+		(property "Footprint" "CRGM Passive:C_0603_1608Metric"
 			(at 86.0552 71.12 0)
 			(effects
@@
 			)
 		)
-		(property "Footprint" "Capacitor_SMD:C_0603_1608Metric"
+		(property "Footprint" "CRGM Passive:C_0603_1608Metric"
 			(at 55.5752 71.12 0)
 			(effects
@@
 			)
 		)
-		(property "Footprint" "Capacitor_SMD:C_0603_1608Metric"
+		(property "Footprint" "CRGM Passive:C_0603_1608Metric"
 			(at 102.5652 71.12 0)
 			(effects
@@
 			)
 		)
-		(property "Footprint" "Capacitor_SMD:C_0603_1608Metric"
+		(property "Footprint" "CRGM Passive:C_0603_1608Metric"
 			(at 70.8152 71.12 0)
 			(effects

Commit message: Added renders and aligned connectors
Added renders
Aligned connectors to grid
Added dimensions
Fixed part numbers and values
Other:
- title: Client Hardware -> Client
Changed lines of the file:
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@@
 	(paper "A4")
 	(title_block
-		(title "Client Hardware")
+		(title "Client")
 		(date "<<release-date>>")
 		(rev "<<tag>>")

Commit message: Added RF connector; re-placed and re-routed
Parts:
- removed C13, C14, C15, C16: 0.1uF, CRGM Passive:C_0603_1608Metric, symbol Device:C
- removed D1, D2, D3, D4: WS2812B-2020, CRGM Passive:LED_WS2812B-2020_PLCC4_2.0x2.0mm, symbol LED:WS2812B-2020
Connections:
- no-connect marks 1 -> 0
Other:
- note removed: "Status LEDs"
- title: Client -> Aquarius Client
