File: pcb/power.kicad_sch (KiCad schematic)
At the start: 21 parts, among them U5 LM66200DRLR, U6 LM66200DRLR, U7 LD1117S33TR

Commit message: Change schematic name
Other:
- title: Relay Module -> Client
Changed lines of the file:
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@@
 	(paper "A4")
 	(title_block
-		(title "Relay Module")
-		(date "2025-03-22")
-		(rev "1.0")
+		(title "Client")
+		(date "<<release-date>>")
+		(rev "<<tag>>")
 		(company "CRG Makes")
-		(comment 1 "Aquarius")
+		(comment 1 "<<hash>>")
 	)
 	(rectangle

Commit message: Updated project name and properties
Other:
- title: Client -> Client Hardware
Changed lines of the file:
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@@
 	(paper "A4")
 	(title_block
-		(title "Client")
+		(title "Client Hardware")
 		(date "<<release-date>>")
 		(rev "<<tag>>")

Commit message: Switch cap/res to CRGM footprint
Parts:
- C7, C8: footprint Capacitor_SMD:C_0603_1608Metric -> CRGM Passive:C_0603_1608Metric
- R8, R9: footprint Resistor_SMD:R_0603_1608Metric -> CRGM Passive:R_0603_1608Metric
Changed lines of the file:
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@@
 			)
 		)
-		(property "Footprint" "Resistor_SMD:R_0603_1608Metric"
+		(property "Footprint" "CRGM Passive:R_0603_1608Metric"
 			(at 142.24 34.29 0)
 			(effects
@@
 			)
 		)
-		(property "Footprint" "Capacitor_SMD:C_0603_1608Metric"
+		(property "Footprint" "CRGM Passive:C_0603_1608Metric"
 			(at 33.9852 87.63 0)
 			(effects
@@
 			)
 		)
-		(property "Footprint" "Capacitor_SMD:C_0603_1608Metric"
+		(property "Footprint" "CRGM Passive:C_0603_1608Metric"
 			(at 56.8452 87.63 0)
 			(effects
@@
 			)
 		)
-		(property "Footprint" "Resistor_SMD:R_0603_1608Metric"
+		(property "Footprint" "CRGM Passive:R_0603_1608Metric"
 			(at 130.81 34.29 0)
 			(effects

Commit message: Added renders and aligned connectors
Added renders
Aligned connectors to grid
Added dimensions
Fixed part numbers and values
Parts:
- C7, C8: MF Samsung -> (none); MN (none) -> Samsung
- D7, D8: footprint LED_SMD:LED_0603_1608Metric -> CRG Makes:LED_0603_1608Metric
- U7: LCSC_PN C86781 -> (none); MF STMicroeletronics -> (none); MN (none) -> STMicroeletronics
Other:
- title: Client Hardware -> Client
Changed lines of the file:
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@@
 	(paper "A4")
 	(title_block
-		(title "Client Hardware")
+		(title "Client")
 		(date "<<release-date>>")
 		(rev "<<tag>>")
@@
 			)
 		)
-		(property "MF" "Samsung"
+		(property "MPN" "CL10B104KO8NNNC"
 			(at 33.02 83.82 0)
 			(effects
@@
 			)
 		)
-		(property "MPN" "CL10B104KO8NNNC"
+		(property "LCSC" "C66501"
 			(at 33.02 83.82 0)
 			(effects
@@
 			)
 		)
-		(property "LCSC" "C66501"
+		(property "Mouser" "187-CL10B104KO8NNNC"
 			(at 33.02 83.82 0)
 			(effects
@@
 			)
 		)
-		(property "Mouser" "187-CL10B104KO8NNNC"
+		(property "Digikey" "1276-1005-2-ND"
 			(at 33.02 83.82 0)
 			(effects
@@
 			)
 		)
-		(property "Digikey" "1276-1005-2-ND"
+		(property "MN" "Samsung"
 			(at 33.02 83.82 0)
 			(effects
@@
 			)
 		)
-		(property "Footprint" "LED_SMD:LED_0603_1608Metric"
+		(property "Footprint" "CRG Makes:LED_0603_1608Metric"
 			(at 142.24 41.91 0)
 			(effects
@@
 			)
 		)
-		(property "MF" "Samsung"
+		(property "MN" "Samsung"
 			(at 55.88 83.82 0)
 			(effects
@@
 			)
 		)
-		(property "LCSC_PN" "C86781"
-			(at 44.45 78.74 0)
-			(effects
-				(font
-					(size 1.27 1.27)
-				)
-				(hide yes)
-			)
-		)
-		(property "MF" "STMicroeletronics"
+		(property "MN" "STMicroeletronics"
 			(at 44.45 78.74 0)
 			(effects
@@
 			)
 		)
-		(property "Footprint" "LED_SMD:LED_0603_1608Metric"
+		(property "Footprint" "CRG Makes:LED_0603_1608Metric"
 			(at 130.81 41.91 0)
 			(effects

Commit message: Added RF connector; re-placed and re-routed
Parts:
- removed C8: 10uF, CRGM Passive:C_0603_1608Metric, symbol Device:C_Small
- removed TP25: ~, CRGM Mechanical:TestPoint_Pad_D1.0mm, symbol Connector:TestPoint
- removed U7: LD1117S33TR, CRGM Power:SOT230P700X180-4N, symbol Regulator_Linear:LD1117S33TR_SOT223
- added C17, C18: 10uF, CRGM Passive:C_0603_1608Metric, symbol Device:C_Small
- added TP41: ~, CRGM Mechanical:TestPoint_Pad_D1.0mm, symbol Connector:TestPoint
- added U9: AZ1084-3.3, CRGM Power:TO-252-2, symbol CRGM Power:AZ1084-3.3
Connections:
- net +5V: now also U9.3 (VI)
- net GND: now also C17.2, C18.2, U9.1 (GND)
- net LDO_V33: now also C17.1, C18.1, TP41.1, U9.2 (VO)
Other:
- title: Client -> Aquarius Client
- moved on the sheet: C7

Commit message: Updated part attributes for consistency
Parts:
- C17, C18, C7: Tolerance (none) -> 10%
- R8: Digikey 541-3993-2-ND -> CR0603-JW-472ELFTR-ND; Mouser 71-CRCW06034K70JNEAC -> 652-CR0603-JW-472ELF; Tolerance (none) -> 5%
- R9: Digikey 541-3991-2-ND -> CR0603-JW-102ELFTR-ND; MN Vishay -> FOJAN; MPN CRCW06031K00FKEA -> FRC0603J102 TS; Mouser 71-CRCW06031K00JNEAC -> 652-CR0603-JW-102ELF; Tolerance (none) -> 5%
Changed lines of the file:
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@@
 			)
 		)
-		(property "Datasheet" "~"
+		(property "Datasheet" "https://bourns.com/docs/product-datasheets/cr.pdf?sfvrsn=574d41f6_14"
 			(at 142.24 34.29 0)
 			(effects
@@
 			)
 		)
-		(property "Description" "Resistor, small symbol"
+		(property "Description" "Thick Film Resistors - SMD 1/10Watt 1Kohms 5%"
 			(at 142.24 34.29 0)
 			(effects
@@
 			)
 		)
-		(property "MN" "Vishay"
+		(property "MN" "FOJAN"
 			(at 142.24 34.29 0)
 			(effects
@@
 			)
 		)
-		(property "MPN" "CRCW06031K00FKEA"
+		(property "MPN" "FRC0603J102 TS"
 			(at 142.24 34.29 0)
 			(effects
@@
 			)
 		)
-		(property "Mouser" "71-CRCW06031K00JNEAC"
+		(property "Mouser" "652-CR0603-JW-102ELF"
 			(at 142.24 34.29 0)
 			(effects
@@
 			)
 		)
-		(property "Digikey" "541-3991-2-ND"
+		(property "Digikey" "CR0603-JW-102ELFTR-ND"
 			(at 142.24 34.29 0)
 			(effects
@@
 			)
 		)
+		(property "Tolerance" "5%"
+			(at 142.24 34.29 0)
+			(effects
+				(font
+					(size 1.27 1.27)
+				)
+				(hide yes)
+			)
+		)
 		(pin "1"
 		)
@@
 			)
 		)
+		(property "Tolerance" "10%"
+			(at 54.61 87.63 0)
+			(effects
+				(font
+					(size 1.27 1.27)
+				)
+				(hide yes)
+			)
+		)
 		(pin "2"
 		)
@@
 			)
 		)
+		(property "Tolerance" "10%"
+			(at 31.75 87.63 0)
+			(effects
+				(font
+					(size 1.27 1.27)
+				)
+				(hide yes)
+			)
+		)
 		(pin "1"
 		)
@@
 			)
 		)
-		(property "Datasheet" "~"
+		(property "Datasheet" "https://bourns.com/docs/product-datasheets/cr.pdf?sfvrsn=574d41f6_14"
 			(at 130.81 34.29 0)
 			(effects
@@
 			)
 		)
-		(property "Description" "Resistor, small symbol"
+		(property "Description" "Thick Film Resistors - SMD 1/10Watt 4.7Kohms 5%"
 			(at 130.81 34.29 0)
 			(effects
@@
 			)
 		)
-		(property "Mouser" "71-CRCW06034K70JNEAC"
+		(property "Mouser" "652-CR0603-JW-472ELF"
 			(at 130.81 34.29 0)
 			(effects
@@
 			)
 		)
-		(property "Digikey" "541-3993-2-ND"
+		(property "Digikey" "CR0603-JW-472ELFTR-ND"
 			(at 130.81 34.29 0)
 			(effects
@@
 			)
 		)
+		(property "Tolerance" "5%"
+			(at 130.81 34.29 0)
+			(effects
+				(font
+					(size 1.27 1.27)
+				)
+				(hide yes)
+			)
+		)
 		(pin "1"
 		)
@@
 			(at 62.23 87.63 0)
 			(effects
+				(font
+					(size 1.27 1.27)
+				)
+				(hide yes)
+			)
+		)
+		(property "Tolerance" "10%"
+			(at 62.23 87.63 0)
+			(effects
