File: pcb/power.kicad_sch (KiCad schematic)
At the start: 22 parts, among them U5 LM66200DRLR, U6 LM66200DRLR, U9 AZ1084-3.3

Commit message: Updated LED footprint
Parts:
- D7, D8: footprint CRG Makes:LED_0603_1608Metric -> CRGM Passive:LED_0603_1608Metric
Changed lines of the file:
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@@
 			)
 		)
-		(property "Footprint" "CRG Makes:LED_0603_1608Metric"
+		(property "Footprint" "CRGM Passive:LED_0603_1608Metric"
 			(at 142.24 41.91 0)
 			(effects
@@
 			)
 		)
-		(property "Footprint" "CRG Makes:LED_0603_1608Metric"
+		(property "Footprint" "CRGM Passive:LED_0603_1608Metric"
 			(at 130.81 41.91 0)
 			(effects
