File: pcb/Archive/env-module.kicad_sch (KiCad schematic)
At the start: 8 parts

Commit message: Added interfaces and fully routed PCB
Parts:
- H1, H2, H3, H4: value ~ -> MountingHole; footprint CRGM Mechanical:MountingHole_3.2mm_M3_Pad_Via -> (none)
- LOGO1: value ~ -> (none); footprint CRGM Logos:CRGM Logo 5mm -> CRGM Logos:CRGM Logo 10mm; now in the parts list
- LOGO2, LOGO3: value ~ -> (none); now in the parts list
- LOGO4: value ~ -> Logo_Open_Hardware_Small; footprint Symbol:OSHW-Logo_5.7x6mm_SilkScreen -> (none)
Changed lines of the file:
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@@
 		(fields_autoplaced yes)
 		(property "Reference" "H1"
-			(at 151.13 170.1799 0)
+			(at 151.13 170.2378 0)
 			(effects
 				(font
@@
 			)
 		)
-		(property "Value" "~"
-			(at 151.13 172.7199 0)
-			(effects
-				(font
-					(size 1.27 1.27)
-				)
-				(justify left)
-				(hide yes)
-			)
-		)
-		(property "Footprint" "CRGM Mechanical:MountingHole_3.2mm_M3_Pad_Via"
+		(property "Value" "MountingHole"
+			(at 157.6213 172.6621 0)
+			(effects
+				(font
+					(size 1.27 1.27)
+				)
+			)
+		)
+		(property "Footprint" ""
 			(at 148.59 171.45 0)
 			(effects
@@
 			)
 		)
-		(property "MPN" ""
-			(at 148.59 171.45 0)
-			(effects
-				(font
-					(size 1.27 1.27)
-				)
-			)
-		)
 		(instances
 			(project "relay-module"
@@
 		(unit 1)
 		(exclude_from_sim no)
-		(in_bom no)
+		(in_bom yes)
 		(on_board yes)
 		(dnp no)
@@
 			)
 		)
-		(property "Value" "~"
+		(property "Value" ""
 			(at 258.064 170.18 0)
 			(effects
@@
 		)
 		(property "Footprint" "CRGM Logos:Aquarius Logo 5mm"
-			(at 261.874 178.308 0)
+			(at 262.636 183.134 0)
 			(effects
 				(font
@@
 			)
 		)
-		(property "MPN" ""
-			(at 260.35 175.26 0)
-			(effects
-				(font
-					(size 1.27 1.27)
-				)
-			)
-		)
-		(property "LCSC" ""
-			(at 260.35 175.26 0)
-			(effects
-				(font
-					(size 1.27 1.27)
-				)
-				(hide yes)
-			)
-		)
-		(property "Digikey" ""
-			(at 260.35 175.26 0)
-			(effects
-				(font
-					(size 1.27 1.27)
-				)
-				(hide yes)
-			)
-		)
-		(property "Mouser" ""
-			(at 260.35 175.26 0)
-			(effects
-				(font
-					(size 1.27 1.27)
-				)
-				(hide yes)
-			)
-		)
 		(instances
 			(project ""
@@
 		(fields_autoplaced yes)
 		(property "Reference" "H3"
-			(at 151.13 180.3399 0)
+			(at 151.13 180.3978 0)
 			(effects
 				(font
@@
 			)
 		)
-		(property "Value" "~"
-			(at 151.13 182.8799 0)
-			(effects
-				(font
-					(size 1.27 1.27)
-				)
-				(justify left)
-				(hide yes)
-			)
-		)
-		(property "Footprint" "CRGM Mechanical:MountingHole_3.2mm_M3_Pad_Via"
+		(property "Value" "MountingHole"
+			(at 157.6213 182.8221 0)
+			(effects
+				(font
+					(size 1.27 1.27)
+				)
+			)
+		)
+		(property "Footprint" ""
 			(at 148.59 181.61 0)
 			(effects
@@
 			)
 		)
-		(property "MPN" ""
-			(at 148.59 181.61 0)
-			(effects
-				(font
-					(size 1.27 1.27)
-				)
-			)
-		)
 		(instances
 			(project "relay-module"
@@
 		(at 271.78 175.26 0)
 		(unit 1)
-		(exclude_from_sim yes)
+		(exclude_from_sim no)
 		(in_bom no)
-		(on_board yes)
+		(on_board no)
 		(dnp no)
 		(fields_autoplaced yes)
@@
 			)
 		)
-		(property "Value" "~"
+		(property "Value" "Logo_Open_Hardware_Small"
 			(at 271.78 180.975 0)
 			(effects
@@
 			)
 		)
-		(property "Footprint" "Symbol:OSHW-Logo_5.7x6mm_SilkScreen"
+		(property "Footprint" ""
 			(at 271.78 175.26 0)
 			(effects
@@
 			)
 		)
+		(property "Sim.Enable" "0"
+			(at 278.6935 174.625 0)
+			(effects
+				(font
+					(size 1.27 1.27)
+				)
+			)
+		)
 		(instances
 			(project ""
@@
 		(fields_autoplaced yes)
 		(property "Reference" "H2"
-			(at 151.13 175.2599 0)
+			(at 151.13 175.3178 0)
 			(effects
 				(font
@@
 			)
 		)
-		(property "Value" "~"
-			(at 151.13 177.7999 0)
-			(effects
-				(font
-					(size 1.27 1.27)
-				)
-				(justify left)
-				(hide yes)
-			)
-		)
-		(property "Footprint" "CRGM Mechanical:MountingHole_3.2mm_M3_Pad_Via"
+		(property "Value" "MountingHole"
+			(at 157.6213 177.7421 0)
+			(effects
+				(font
+					(size 1.27 1.27)
+				)
+			)
+		)
+		(property "Footprint" ""
 			(at 148.59 176.53 0)
 			(effects
@@
 			)
 		)
-		(property "MPN" ""
-			(at 148.59 176.53 0)
-			(effects
-				(font
-					(size 1.27 1.27)
-				)
-			)
-		)
 		(instances
 			(project "relay-module"
@@
 		(unit 1)
 		(exclude_from_sim no)
-		(in_bom no)
+		(in_bom yes)
 		(on_board yes)
 		(dnp no)
@@
 			)
 		)
-		(property "Value" "~"
+		(property "Value" ""
 			(at 248.92 173.99 0)
 			(effects
@@
 			)
 		)
-		(property "Footprint" "CRGM Logos:CRGM Logo 5mm"
+		(property "Footprint" "CRGM Logos:CRGM Logo 10mm"
 			(at 248.92 182.118 0)
 			(effects
@@
 			)
 		)
-		(property "LCSC" ""
-			(at 248.92 173.99 0)
-			(effects
-				(font
-					(size 1.27 1.27)
-				)
-				(hide yes)
-			)
-		)
-		(property "Digikey" ""
-			(at 248.92 173.99 0)
-			(effects
-				(font
-					(size 1.27 1.27)
-				)
-				(hide yes)
-			)
-		)
-		(property "Mouser" ""
-			(at 248.92 173.99 0)
-			(effects
-				(font
-					(size 1.27 1.27)
-				)
-				(hide yes)
-			)
-		)
 		(instances
 			(project ""
@@
 		(unit 1)
 		(exclude_from_sim no)
-		(in_bom no)
+		(in_bom yes)
 		(on_board yes)
 		(dnp no)
@@
 			)
 		)
-		(property "Value" "~"
+		(property "Value" ""
 			(at 235.204 170.18 0)
 			(effects
@@
 		)
 		(property "Footprint" "CRGM Logos:Aquarius Logo 5mm"
-			(at 239.014 178.308 0)
+			(at 239.776 183.134 0)
 			(effects
 				(font
@@
 			)
 		)
-		(property "MPN" ""
-			(at 237.49 175.26 0)
-			(effects
-				(font
-					(size 1.27 1.27)
-				)
-			)
-		)
-		(property "LCSC" ""
-			(at 237.49 175.26 0)
-			(effects
-				(font
-					(size 1.27 1.27)
-				)
-				(hide yes)
-			)
-		)
-		(property "Digikey" ""
-			(at 237.49 175.26 0)
-			(effects
-				(font
-					(size 1.27 1.27)
-				)
-				(hide yes)
-			)
-		)
-		(property "Mouser" ""
-			(at 237.49 175.26 0)
-			(effects
-				(font
-					(size 1.27 1.27)
-				)
-				(hide yes)
-			)
-		)
 		(instances
 			(project "servo-module"
@@
 		(fields_autoplaced yes)
 		(property "Reference" "H4"
-			(at 151.13 185.4199 0)
+			(at 151.13 185.4778 0)
 			(effects
 				(font
@@
 			)
 		)
-		(property "Value" "~"
-			(at 151.13 187.9599 0)
-			(effects
-				(font
-					(size 1.27 1.27)
-				)
-				(justify left)
-				(hide yes)
-			)
-		)
-		(property "Footprint" "CRGM Mechanical:MountingHole_3.2mm_M3_Pad_Via"
+		(property "Value" "MountingHole"
+			(at 157.6213 187.9021 0)
+			(effects
+				(font
+					(size 1.27 1.27)
+				)
+			)
+		)
+		(property "Footprint" ""
 			(at 148.59 186.69 0)
 			(effects
@@
 			)
 		)
-		(property "MPN" ""
-			(at 148.59 186.69 0)
-			(effects
-				(font
-					(size 1.27 1.27)
-				)
-			)
-		)
